File: nrfdevboard.kicad_sch (KiCad schematic)
At the start: 17 parts, among them J1 Conn_01x07_Pin, J2 Conn_01x07_Pin, P1 Straddle_USB_type_c, U1 MDBT50Q-P1MV2, U3 AP2112K-3.3TRG1, Y1 O_32.768kHz

Commit message: Routing done (outside USB) + added some more pins
Parts:
- added J3: 3_tht_side, Connector_PinHeader_2.54mm:PinHeader_1x03_P2.54mm_Vertical, symbol Connector:Conn_01x03_Pin
- added J4: 2_tht_top, Connector_PinHeader_2.54mm:PinHeader_1x02_P2.54mm_Vertical, symbol Connector:Conn_01x02_Pin
- added J5: 1_tht_top, Connector_PinHeader_2.54mm:PinHeader_1x01_P2.54mm_Vertical, symbol Connector:Conn_01x01_Pin
- added TP1: TestPoint, symbol Connector:TestPoint
- J1: value Conn_01x07_Pin -> 7_print_front
- J2: value Conn_01x07_Pin -> 7_pin_back
Connections:
- net +3.3V: now also J1.7 (Pin_7)
- net GND: now also J4.2 (Pin_2); no longer J1.7 (Pin_7)
- net PIN8: now also U1.27 (P0.11/TRACEDATA2); no longer U1.40 (P0.18/nRESET)
- net VBUS: now also J4.1 (Pin_1)
- net PIN15: now reaches U1.36 (P0.14)
- net PIN15: now also J3.3 (Pin_3)
- net PIN16: now reaches U1.38 (P0.16)
- net PIN16: now also J3.2 (Pin_2)
- net PIN17: now reaches U1.43 (P0.21)
- net PIN17: now also J3.1 (Pin_1)
- new net PIN20: J5.1 (Pin_1), U1.40 (P0.18/nRESET)
- no-connect marks 48 -> 44

Commit message: Basics done. Will need to optimise double check DFM before manufacturing
Connections:
- net PIN10: now also U1.27 (P0.11/TRACEDATA2); no longer U1.25 (P1.08)
- net PIN8: now also U1.45 (PO23); no longer U1.27 (P0.11/TRACEDATA2)
- net D+_r renamed mcu_D+
- net D-_r renamed mcu_D-
Changed lines of the file:
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@@
-	)
-	(no_connect
-		(at 121.92 147.32)
 	)
 	(no_connect
@@
 	)
 	(no_connect
+		(at 147.32 181.61)
+	)
+	(no_connect
 		(at 43.18 92.71)
 	)
@@
 	(wire
 		(pts
+			(xy 120.65 147.32) (xy 121.92 147.32)
+		)
+		(stroke
+			(width 0)
+			(type default)
+		)
+	)
+	(wire
+		(pts
 			(xy 43.18 41.91) (xy 49.53 41.91)
 		)
@@
 		(pts
 			(xy 68.58 128.27) (xy 68.58 125.73)
-		)
-		(stroke
-			(width 0)
-			(type default)
-		)
-	)
-	(wire
-		(pts
-			(xy 147.32 181.61) (xy 147.32 184.15)
 		)
 		(stroke
@@
 		)
 	)
-	(label "D-_r"
+	(label "mcu_D-"
 		(at 135.89 113.03 90)
 		(effects
@@
 		)
 	)
-	(label "D+_r"
+	(label "mcu_D+"
 		(at 138.43 113.03 90)
 		(effects
@@
 	(global_label "PIN10"
 		(shape input)
-		(at 147.32 184.15 270)
-		(fields_autoplaced yes)
-		(effects
-			(font
-				(size 1.27 1.27)
-			)
-			(justify right)
-		)
-		(property "Intersheetrefs" "${INTERSHEET_REFS}"
-			(at 147.32 192.2604 90)
+		(at 152.4 184.15 270)
+		(fields_autoplaced yes)
+		(effects
+			(font
+				(size 1.27 1.27)
+			)
+			(justify right)
+		)
+		(property "Intersheetrefs" "${INTERSHEET_REFS}"
+			(at 152.4 192.2604 90)
 			(effects
 				(font
@@
 	(global_label "PIN8"
 		(shape input)
-		(at 152.4 184.15 270)
-		(fields_autoplaced yes)
-		(effects
-			(font
-				(size 1.27 1.27)
-			)
-			(justify right)
-		)
-		(property "Intersheetrefs" "${INTERSHEET_REFS}"
-			(at 152.4 191.1909 90)
-			(effects
-				(font
+		(at 120.65 147.32 180)
+		(fields_autoplaced yes)
+		(effects
+			(font
+				(size 1.27 1.27)
+			)
+			(justify right)
+		)
+		(property "Intersheetrefs" "${INTERSHEET_REFS}"
+			(at 113.6091 147.32 0)
+			(effects
+				(font

Commit message: Clearing up DRC errors (part 1)
Parts:
- H1: footprint MountingHole:MountingHole_2.2mm_M2 -> TH-1-CC:PDB_MountingHole_left_2.2mm_M2
- H3: footprint MountingHole:MountingHole_2.2mm_M2_Pad -> TH-1-CC:PDB_MountingHole_right_2.2mm_M2_Pad
Changed lines of the file:
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@@
 			)
 		)
-		(property "Footprint" "MountingHole:MountingHole_2.2mm_M2_Pad"
+		(property "Footprint" "TH-1-CC:PDB_MountingHole_right_2.2mm_M2_Pad"
 			(at 219.71 63.5 0)
 			(effects
@@
 			)
 		)
-		(property "Footprint" "MountingHole:MountingHole_2.2mm_M2"
+		(property "Footprint" "TH-1-CC:PDB_MountingHole_left_2.2mm_M2"
 			(at 222.25 77.47 0)
 			(effects
