File: nrfdevboard.kicad_pcb (KiCad board)
At the start: 4 copper layers, 26 x 26.2 mm, 20 parts, among them J1 7_print_front, J2 7_pin_back, J3 3_tht_side, J4 2_tht_top, J5 1_tht_top, P1 Straddle_USB_type_c, U1 MDBT50Q-P1MV2, U3 AP2112K-3.3TRG1, Y1 O_32.768kHz

Commit message: Fixed remaining DRC errors
Parts:
- P1: footprint TH-1-CC_footprints:USBC -> TH-1-CC:USBC
Routing:
- net unconnected-(U1B-DCCH-Pad31): track 1.22 -> 0.00 mm, vias 1 -> 0
- net GND: track 41.4 -> 42.6 mm, vias 33 -> 34
- net VBUS: track 41.2 -> 41.6 mm, vias 2 -> 1
Changed lines of the file:
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@@
 			(at 0 -3.15 0)
 			(layer "F.SilkS")
+			(hide yes)
 			(effects
 				(font
@@
 		)
 	)
-	(footprint "TH-1-CC_footprints:USBC"
+	(footprint "TH-1-CC:USBC"
 		(layer "F.Cu")
 		(at 89.15 115.35)
@@
 			(unlocked yes)
 			(layer "F.SilkS")
-			(hide yes)
 			(effects
 				(font
@@
 			(pinfunction "GND")
 			(pintype "passive")
+			(solder_mask_margin -0.02)
 		)
 		(pad "A2" smd roundrect
@@
 			(pinfunction "TX1+")
 			(pintype "bidirectional+no_connect")
+			(solder_mask_margin -0.02)
 		)
 		(pad "A3" smd roundrect
@@
 			(pinfunction "TX1-")
 			(pintype "bidirectional+no_connect")
+			(solder_mask_margin -0.02)
 		)
 		(pad "A4" smd roundrect
@@
 			(pinfunction "VBUS")
 			(pintype "passive")
+			(solder_mask_margin -0.02)
 		)
 		(pad "A5" smd roundrect
@@
 			(pinfunction "CC")
 			(pintype "bidirectional")
+			(solder_mask_margin -0.02)
 		)
 		(pad "A6" smd roundrect
@@
 			(pinfunction "D+")
 			(pintype "bidirectional")
+			(solder_mask_margin -0.02)
 		)
 		(pad "A7" smd roundrect
@@
 			(pinfunction "D-")
 			(pintype "bidirectional")
+			(solder_mask_margin -0.02)
 		)
 		(pad "A8" smd roundrect
@@
 			(pinfunction "SBU1")
 			(pintype "bidirectional+no_connect")
+			(solder_mask_margin -0.02)
 		)
 		(pad "A9" smd roundrect
@@
 			(pinfunction "VBUS")
 			(pintype "passive")
+			(solder_mask_margin -0.02)
 		)
 		(pad "A10" smd roundrect
@@
 			(pinfunction "RX2-")
 			(pintype "bidirectional+no_connect")
+			(solder_mask_margin -0.02)
 		)
 		(pad "A11" smd roundrect
@@
 			(pinfunction "RX2+")
 			(pintype "bidirectional+no_connect")
+			(solder_mask_margin -0.02)
 		)
 		(pad "A12" smd roundrect
@@
 			(pinfunction "GND")
 			(pintype "passive")
+			(solder_mask_margin -0.02)
 		)
 		(pad "B1" smd roundrect
@@
 			(pinfunction "GND")
 			(pintype "passive")
+			(solder_mask_margin -0.02)
 		)
 		(pad "B2" smd roundrect
@@
 			(pinfunction "TX2+")
 			(pintype "bidirectional+no_connect")
+			(solder_mask_margin -0.02)
 		)
 		(pad "B3" smd roundrect
@@
 			(pinfunction "TX2-")
 			(pintype "bidirectional+no_connect")
+			(solder_mask_margin -0.02)
 		)
 		(pad "B4" smd roundrect
@@
 			(pinfunction "VBUS")
 			(pintype "passive")
+			(solder_mask_margin -0.02)
 		)
 		(pad "B5" smd roundrect
@@
 			(pinfunction "VCONN")
 			(pintype "bidirectional+no_connect")
+			(solder_mask_margin -0.02)
 		)
 		(pad "B8" smd roundrect
@@
 			(pinfunction "SBU2")
 			(pintype "bidirectional+no_connect")
+			(solder_mask_margin -0.02)
 		)
 		(pad "B9" smd roundrect
@@
 			(pinfunction "VBUS")
 			(pintype "passive")
+			(solder_mask_margin -0.02)
 		)
 		(pad "B10" smd roundrect
@@
 			(pinfunction "RX1-")
 			(pintype "bidirectional+no_connect")
+			(solder_mask_margin -0.02)
 		)
 		(pad "B11" smd roundrect
@@
 			(pinfunction "RX1+")
 			(pintype "bidirectional+no_connect")
+			(solder_mask_margin -0.02)
 		)
 		(pad "B12" smd roundrect
@@
 			(pinfunction "GND")
 			(pintype "passive")
+			(solder_mask_margin -0.02)
 		)
 		(pad "S1" smd roundrect
@@
 			(pinfunction "SHIELD")
 			(pintype "passive")
+			(solder_mask_margin -0.02)
 		)
 		(pad "S1" smd roundrect
@@
 			(pinfunction "SHIELD")
 			(pintype "passive")
+			(solder_mask_margin -0.02)
 		)
 		(embedded_fonts no)
-		(model "${KIPRJMOD}/non-licence/1054440001.stp"
-			(offset
-				(xyz 4 11 -0.5)
-			)
-			(scale
-				(xyz 1 1 1)
-			)
-			(rotate
-				(xyz 90 -0 -0)
-			)
-		)
 	)
 	(footprint "Resistor_SMD:R_0603_1608Metric"
@@
 		(tags "mountinghole M2")
 		(property "Reference" "H3"
-			(at 0 -3.15 0)
+			(at -0.7 -0.975 0)
 			(layer "F.SilkS")
+			(hide yes)
 			(effects
 				(font
@@
 	)
 	(segment
+		(start 90.875 121.45)
+		(end 90.875 120.325)
+		(width 0.3)
+		(layer "F.Cu")
+		(net 1)
+	)
+	(segment
 		(start 99.45 119.55)
 		(end 100.3 118.7)
@@
 	)
 	(segment
+		(start 90.875 120.325)
+		(end 90.85 120.3)
+		(width 0.3)
+		(layer "F.Cu")
+		(net 1)
+	)
+	(segment
 		(start 95.75 121.65)
 		(end 95.7 121.6)
@@
 	)
 	(via
+		(at 90.875 121.45)
+		(size 0.65)
+		(drill 0.35)
+		(layers "F.Cu" "B.Cu")
+		(net 1)
+	)
+	(via
 		(at 101.1 116.875)
 		(size 0.65)
@@
 	)
 	(segment
-		(start 94.45 117.05)
-		(end 94.8 117.4)
+		(start 95 117.6)
+		(end 95.05 117.65)
 		(width 0.3)
 		(layer "F.Cu")
@@
 	)
 	(segment
-		(start 95.05 117.65)
-		(end 94.8 117.4)
-		(width 0.5)
-		(layer "F.Cu")
-		(net 3)
-	)
-	(segment
 		(start 101.7666 117.7)
 		(end 101.2 117.7)
@@
 	)
 	(segment
+		(start 95.05 117.65)
+		(end 99 117.65)
+		(width 0.3)
+		(layer "F.Cu")
+		(net 3)
+	)
+	(segment
+		(start 94.45 117.05)
+		(end 95 117.6)
+		(width 0.3)
+		(layer "F.Cu")
+		(net 3)
+	)
+	(segment
 		(start 91.074 117.876)
 		(end 91.95 117)
@@
 	)
 	(segment
+		(start 89.675 117.876)
+		(end 91.074 117.876)
+		(width 0.3)
+		(layer "F.Cu")
+		(net 3)
+	)
+	(segment
 		(start 91.95 117)
 		(end 91.95 116.1)
@@
 	)
 	(segment
-		(start 99 117.65)
-		(end 95.05 117.65)
-		(width 0.5)
-		(layer "F.Cu")
-		(net 3)
-	)
-	(segment
 		(start 98.1 121.6)
 		(end 99.176 120.524)
@@
 	(segment
 		(start 88.266 117.876)
-		(end 91.074 117.876)
+		(end 89.675 117.876)
 		(width 0.3)
 		(layer "F.Cu")
@@
 	)
 	(via
-		(at 94.8 117.4)
+		(at 94.95 117.65)
 		(size 0.65)
 		(drill 0.35)
 		(layers "F.Cu" "B.Cu")
-		(free yes)
-		(tenting none)
-		(net 3)
-	)
-	(via
-		(at 89.65 117.875564)
-		(size 0.6)
-		(drill 0.3)
-		(layers "F.Cu" "B.Cu")
 		(net 3)
 	)
@@
 	)
 	(segment
-		(start 94.324436 117.875564)
-		(end 94.8 117.4)
-		(width 0.3)
-		(layer "B.Cu")
-		(net 3)
-	)
-	(segment
-		(start 94.45 117.05)
-		(end 94.8 117.4)
+		(start 91.95 117)
+		(end 91.075 117.875)
 		(width 0.3)
 		(layer "B.Cu")
@@
 	(segment
 		(start 89.65 117.875564)
-		(end 94.324436 117.875564)
+		(end 94.724436 117.875564)
 		(width 0.3)
 		(layer "B.Cu")
@@
 	)
 	(segment
-		(start 94.45 116.1)
-		(end 94.45 117.05)
+		(start 94.724436 117.875564)
+		(end 94.95 117.65)
 		(width 0.3)
 		(layer "B.Cu")
@@
 	)
 	(segment
-		(start 91.95 117)
-		(end 91.075 117.875)
+		(start 88.626 117.876)
+		(end 88.266 117.876)
 		(width 0.3)
 		(layer "B.Cu")
@@
 	)
 	(segment
-		(start 88.626 117.876)
-		(end 88.266 117.876)
+		(start 94.95 117.65)
+		(end 95 117.6)
 		(width 0.3)
 		(layer "B.Cu")
@@
 	)
 	(segment
+		(start 94.45 116.1)
+		(end 94.45 117.05)
+		(width 0.3)
+		(layer "B.Cu")
+		(net 3)
+	)
+	(segment
+		(start 94.45 117.05)
+		(end 95 117.6)
+		(width 0.3)
+		(layer "B.Cu")
+		(net 3)
+	)
+	(segment
 		(start 90.975 117.875)
 		(end 89.65 117.875564)
@@
 	)
 	(segment
-		(start 95.216732 123.800002)
-		(end 94.733365 123.316635)
-		(width 0.3)
-		(layer "F.Cu")
-		(net 23)
-	)
-	(segment
-		(start 95.75 123.800002)
-		(end 95.216732 123.800002)
-		(width 0.3)
-		(layer "F.Cu")
-		(net 23)
-	)
-	(via
-		(at 94.733365 123.316635)
-		(size 0.65)
-		(drill 0.35)
-		(layers "F.Cu" "B.Cu")
-		(tenting none)
-		(net 23)
-	)
-	(segment
